File: BLDC_4.kicad_pcb (KiCad board)
At the start: 4 copper layers, 160 x 160 mm, 103 parts, among them J1 RJ45, K1 SERVO, P2 SWD, P4 IN+, P5 IN-, P6 MOTOR1, P7 MOTOR2, P9 MOTOR3, Q1 IRFS7530, Q2 IRFS7530, Q3 IRFS7530, Q4 IRFS7530, Q5 IRFS7530, Q6 IRFS7530, U1 STM32F40X_LQFP64, U2 TC2117, U3 DRV8302, U401 SN65HVD232, X1 MINI-USB-SHIELD-32005-201, X2 8MHz 10ppm

Commit message: ttt
Parts:
- moved R2 190.8 mm to (116.8, 167.6)
- moved C41 189.5 mm to (122.4, 167.6)
- moved R1 189.4 mm to (115.6, 162.6)
- moved C8 182.9 mm to (138.4, 209.6), turned to 180 degrees
- moved C40 167.8 mm to (118.1, 152.4)
- moved C1 167.2 mm to (117.7, 148.6)
- moved C39 159.7 mm to (118.5, 142.2)
- moved C26 159.6 mm to (168.4, 193.0)
- moved C27 159.6 mm to (118.1, 144.8)
- moved C18 157.3 mm to (160.6, 192.8)
- moved C28 157.3 mm to (163.1, 192.8)
- moved C36 157.3 mm to (160.6, 194.2)
- moved C52 157.3 mm to (163.1, 194.2)
- moved R20 157.3 mm to (155.8, 192.3)
- moved R33 157.3 mm to (158.1, 193.8)
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
Commit message: no message
Parts:
- moved C8 155.9 mm to (182.9, 60.1), turned to 270 degrees
- moved C26 147.3 mm to (135.1, 49.5)
- moved C28 144.6 mm to (138.4, 50.3), turned to 90 degrees
- moved C22 143.6 mm to (147.8, 49.5), turned to 180 degrees
- moved C18 143.0 mm to (135.1, 52.1)
- moved C52 142.2 mm to (138.4, 54.1), turned to 90 degrees
- moved C36 141.9 mm to (135.1, 54.6)
- moved C21 139.4 mm to (151.1, 49.5)
- moved R20 135.5 mm to (138.4, 57.9), turned to 90 degrees
- moved R33 134.3 mm to (138.4, 61.0), turned to 90 degrees
- moved C34 133.8 mm to (141.0, 62.2), turned to 180 degrees
- moved C9 131.1 mm to (129.2, 48.3), turned to 180 degrees
- moved C24 126.0 mm to (175.3, 55.9)
- moved C33 123.3 mm to (158.5, 53.3), turned to 180 degrees
- moved C49 122.0 mm to (129.2, 53.3)
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
Commit message: no message
Parts:
- moved C40 103.3 mm to (185.4, 74.0), turned to 270 degrees
- moved C1 103.0 mm to (190.5, 74.0), turned to 270 degrees
- moved R49 83.2 mm to (125.7, 77.5), turned to 270 degrees
- moved R2 79.1 mm to (175.3, 114.3), turned to 90 degrees
- moved R50 77.9 mm to (128.7, 77.8), turned to 270 degrees
- moved C41 76.9 mm to (177.8, 114.3), turned to 90 degrees
- moved C43 75.0 mm to (129.2, 62.2), turned to 0 degrees
- moved R51 75.0 mm to (131.2, 77.8), turned to 270 degrees
- moved R1 74.8 mm to (172.7, 114.3), turned to 270 degrees
- moved C27 74.4 mm to (152.4, 78.7), turned to 180 degrees
- moved C39 74.1 mm to (152.0, 76.2)
- moved R23 73.6 mm to (135.1, 61.0)
- moved C20 72.1 mm to (137.2, 62.7), turned to 90 degrees
- moved R32 71.4 mm to (133.5, 78.2), turned to 270 degrees
- moved R18 69.3 mm to (139.7, 62.7), turned to 270 degrees
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
Commit message: First Commit of Altium Project
Parts:
- J1: footprint Connector_RJ:RJ45_Amphenol_54602-x08_Horizontal -> Connector_RJ:RJ45_Amphenol_RJHSE538X
- moved R24 37.1 mm to (126.2, 58.4)
- moved R27 28.8 mm to (138.4, 79.2), turned to 90 degrees
- moved C14 28.8 mm to (146.1, 102.1), turned to 270 degrees
- moved R18 25.1 mm to (151.6, 40.6), turned to 180 degrees
- moved C22 22.9 mm to (147.8, 40.6)
- moved C23 22.9 mm to (142.2, 39.9), turned to 270 degrees
- moved C30 22.9 mm to (144.8, 39.9), turned to 270 degrees
- moved R17 22.9 mm to (158.8, 40.6)
- moved R21 22.9 mm to (154.9, 40.6)
- moved C11 21.3 mm to (163.1, 90.2), turned to 0 degrees
- moved C21 21.1 mm to (130.8, 57.9), turned to 270 degrees
- moved R28 20.6 mm to (102.1, 100.3), turned to 0 degrees
- moved J1 20.5 mm to (115.6, 119.4)
- moved R54 19.3 mm to (118.8, 104.9)
- moved C10 19.2 mm to (163.1, 95.2), turned to 0 degrees
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Routing:
- net /Mosfet driver/M_L1: track 0.00 -> 49.7 mm, vias 0 -> 2
- net Net-(R20-Pad1): track 0.00 -> 28.0 mm, vias 0 -> 4
- net Net-(C28-Pad2): track 0.00 -> 23.7 mm, vias 0 -> 2
- net Net-(C20-Pad2): track 0.00 -> 20.5 mm, vias 0 -> 3
- net /Mosfet driver/H1_LOW: track 0.00 -> 17.6 mm, vias 0 -> 1
- net /Mosfet driver/M_L3: track 0.00 -> 14.8 mm, vias 0 -> 2
- net /Mosfet driver/H1_VS: track 0.00 -> 13.7 mm, vias 0 -> 1
- net Net-(C36-Pad1): track 0.00 -> 13.5 mm, vias 0 -> 1
- net /Mosfet driver/M_L2: track 0.00 -> 11.9 mm, vias 0 -> 2
- net /Mosfet driver/H2_VS: track 0.00 -> 11.9 mm, vias 0 -> 3
- net /MCU/BR_SO1: track 0.00 -> 11.2 mm, vias 0 -> 2
- net Net-(C29-Pad2): track 0.00 -> 10.9 mm, vias 0 -> 1
- net /MCU/FAULT: track 0.00 -> 10.8 mm, vias 0 -> 1
- net /MCU/SENS3: track 0.00 -> 10.1 mm
- net Net-(C27-Pad1): track 0.00 -> 9.42 mm
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Other:
- copper layers 4 -> 2
- net class Default: clearance 0.1778 -> 0.15; trace_width 0.2032 -> 0.15
- rule trace_clearance: 0.1778 -> 0.15
- rule trace_min: 0.2032 -> 0.15
